Commit message: working rviz robot interaction

File: my_urdf_folder/config/ebamk2.ros2_control.xacro (robot description, xacro)
@@ -38,11 +38,4 @@
                 <state_interface name="velocity"/>
             </joint>
-            <joint name="joint_6">
-                <command_interface name="position"/>
-                <state_interface name="position">
-                  <param name="initial_value">${initial_positions['joint_6']}</param>
-                </state_interface>
-                <state_interface name="velocity"/>
-            </joint>
         </ros2_control>
     </xacro:macro>

Commit message: calibration in python script instead of firmware

File: my_urdf_folder/config/ebamk2.ros2_control.xacro (robot description, xacro)
@@ -38,4 +38,11 @@
                 <state_interface name="velocity"/>
             </joint>
+            <joint name="joint_6">
+                <command_interface name="position"/>
+                <state_interface name="position">
+                  <param name="initial_value">${initial_positions['joint_6']}</param>
+                </state_interface>
+                <state_interface name="velocity"/>
+            </joint>
         </ros2_control>
     </xacro:macro>
